File: VXO_PSU.sch (KiCad schematic (older format))
At the start: 48 parts, among them CON1 BARREL_JACK, P1 CONN_01X02, P10 CONN_02X08, P11 CONN_02X08, P12 BNC, P13 BNC, P2 CONN_02X08, P3 CONN_02X08, P4 CONN_02X08, P5 CONN_02X08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

Commit message: rework to verson 1.1, changing inductors, removing pi output filters
Parts:
- removed L5, L6: 10µH, Inductors_SMD:L_Taiyo-Yuden_NR-40xx, symbol INDUCTOR
- added C24: 4.7µ, Capacitors_SMD:C_1206, symbol C_US
- C23: value CP_US -> 680µF; footprint Capacitors_THT:CP_Radial_D8.0mm_P3.50mm -> Capacitors_THT:CP_Radial_D12.5mm_P5.00mm
- L1: Part Number (none) -> SRR6038-120Y
- L4: value 10µH -> 82µH; footprint Inductors_SMD:L_Taiyo-Yuden_NR-40xx -> MyModules:SRR1260-820M
Connections:
- net +12V: now also C5.1, U1.3 (VO); no longer L4.2
- net +5V: now also C7.1, U3.3 (VO)
- net -12V: now also C6.2, U2.2 (GND)
- net GND: now also C24.2
- net at C1.1, C23.1 (+), L1.1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: now also L4.2, C24.1; no longer D1.1 (K)
- new net: D1.1 (K), L4.1
Other:
- moved on the sheet: C11, C12, C13, C14, C15, C16, C17, C18, C19, C20, C21, C22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

Commit message: fiddly tricks
Parts:
- L2: value 12µH -> 10µH
- L4: Part Number (none) -> SRR1260-820M‎
Changed lines of the file:
@@
 F 2 "Inductors_SMD:L_Taiyo-Yuden_NR-40xx" H 16250 11825 60  0001 C CNN
 F 3 "" H 16250 11825 60  0000 C CNN
-F 4 "SRR6038-120Y" V 16425 11825 60  0000 C CNN "Part Number"
+F 4 "SRR6038-120Y" V 16450 11825 60  0000 C CNN "Part Number"
 	1    16250 11825
 	0    -1   -1   0
@@
 P 16275 10450
 F 0 "L2" V 16175 10450 50  0000 C CNN
-F 1 "12µH" V 16400 10450 50  0000 C CNN
+F 1 "10µH" V 16400 10450 50  0000 C CNN
 F 2 "Inductors_SMD:L_Taiyo-Yuden_NR-40xx" H 16275 10450 60  0001 C CNN
 F 3 "NRS4018T100MDGJ" V 16500 10450 60  0000 C CNN
@@
 F 2 "MyModules:SRR1260-820M" H 14275 11825 60  0001 C CNN
 F 3 "" H 14275 11825 60  0000 C CNN
+F 4 "SRR1260-820M‎" V 14500 11800 60  0000 C CNN "Part Number"
 	1    14275 11825
 	0    -1   -1   0
