File: VXO_PSU.sch (KiCad schematic (older format))
At the start: 48 parts, among them CON1 BARREL_JACK, P1 CONN_01X02, P10 CONN_02X08, P11 CONN_02X08, P12 BNC, P13 BNC, P2 CONN_02X08, P3 CONN_02X08, P4 CONN_02X08, P5 CONN_02X08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

Commit message: added back negative rail pi filter, changed input L footprint
Parts:
- removed C10: 22µF, Capacitors_SMD:C_1206, symbol C_US
- removed L4, L6: 10µH, Inductors_SMD:L_Taiyo-Yuden_NR-40xx, symbol INDUCTOR
- C23: value CP_US -> 220µ
- CON1: Part Number (none) -> ‎EJ508A‎
- L1: footprint Inductors_SMD:L_Taiyo-Yuden_NR-40xx -> MyModules:SRR6038-120Y; Part Number (none) -> SRR6038-120Y
- L2: value 12µH -> 10µH
- P12: Part Number (none) -> 5-1634503-1‎
- U1, U2: value VX078-500 -> VX078012-1000; footprint MyModules:R-78E-0.5 -> MyModules:CONV_VXO78012-1000
- U3: footprint MyModules:R-78E-0.5 -> MyModules:CUI_VXO780XX-500
Connections:
- net +12V: now also C5.1, U1.3 (VO)
- net +5V: now also C7.1, U3.3 (VO)
